Commit message: check mobile franka,can't close

File: assets/robot/franka_description/franka_panda_mobile_xy_tz.urdf (robot description, URDF)
Before this commit: robot panda, 19 links, 18 joints
Links:
- removed link ee_grasp_frame
- removed link ee_link
- removed link grasp_frame
- link panda_hand: geometry collision mesh filename=meshes/collision/hand.obj; visual mesh filename=meshes/visual/hand.obj
Joints:
- removed joint ee_fixed_joint
- removed joint ee_fixed_t
- removed joint ee_grasp_joint
